Commit message: Changed core turning mechanics for the robot, finalized test robot URDF file

File: assets/simple_robot.urdf (robot description, URDF)
Before this commit: robot simple_robot, 3 links, 2 joints
Links:
- removed link left_wheel
- removed link right_wheel
- added link front_indicator, mass 1.0; collision box size=0.1 0.1 0.1; visual box size=0.1 0.1 0.1
- added link front_left_wheel, mass 1.0; collision cylinder length=0.05 radius=0.05; visual cylinder length=0.05 radius=0.05
- added link front_right_wheel, mass 1.0; collision cylinder length=0.05 radius=0.05; visual cylinder length=0.05 radius=0.05
- added link rear_left_wheel, mass 1.0; collision cylinder length=0.05 radius=0.05; visual cylinder length=0.05 radius=0.05
- added link rear_right_wheel, mass 1.0; collision cylinder length=0.05 radius=0.05; visual cylinder length=0.05 radius=0.05
- link base_link: mass 1.0 -> 5.0; geometry collision box size=0.5 0.3 0.1; visual box size=0.5 0.3 0.1
Joints:
- removed joint left_wheel_joint
- removed joint right_wheel_joint
- added joint front_indicator_joint: type fixed, parent base_link, child front_indicator, origin xyz=0 0 0 rpy=0 0 0, axis 0 0 1
- added joint front_left_wheel_joint: type continuous, parent base_link, child front_left_wheel, origin xyz=0.2 0.15 -0.05 rpy=1.57 0 0, axis 0 0 1
- added joint front_right_wheel_joint: type continuous, parent base_link, child front_right_wheel, origin xyz=0.2 -0.15 -0.05 rpy=1.57 0 0, axis 0 0 1
- added joint rear_left_wheel_joint: type continuous, parent base_link, child rear_left_wheel, origin xyz=-0.2 0.15 -0.05 rpy=1.57 0 0, axis 0 0 1
- added joint rear_right_wheel_joint: type continuous, parent base_link, child rear_right_wheel, origin xyz=-0.2 -0.15 -0.05 rpy=1.57 0 0, axis 0 0 1
